Commit message: change front_camera_pivot_joint from fixed type to revolute type, still need tune PID

File: src/ridgeback/ridgeback_description/urdf/accessories/camera_mount.urdf.xacro (robot description, xacro)
@@ -34,9 +34,21 @@
       </visual>
     </link>
-    <joint name="${prefix}_camera_pivot_joint" type="fixed">
+    <joint name="${prefix}_camera_pivot_joint" type="revolute">
       <origin xyz="0.102 0 0.008" rpy="0 ${tilt} 0" />
       <parent link="${prefix}_camera_mount" />
       <child link="${prefix}_camera_beam" />
+      <limit upper="1.57" lower="-1.57" velocity="0.3" effort="10"/>
+       <axis xyz="0 0 1" />
     </joint>
+    <transmission name="turret_trans">
+    <type>transmission_interface/SimpleTransmission</type>
+    <joint name="front_camera_pivot_joint">
+      <hardwareInterface>hardware_interface/PositionJointInterface</hardwareInterface>
+    </joint>
+    <actuator name="turret_motor">
+      <hardwareInterface>hardware_interface/PositionJointInterface</hardwareInterface>
+      <mechanicalReduction>1</mechanicalReduction>
+    </actuator>
+  </transmission>
     <gazebo reference="${prefix}_camera_beam">
       <material>Gazebo/DarkGrey</material>

Commit message: finish turrent

File: src/ridgeback/ridgeback_description/urdf/accessories/camera_mount.urdf.xacro (robot description, xacro)
@@ -18,5 +18,5 @@
       <inertial>
         <origin xyz="0 0 0" rpy="0 0 0" />
-        <mass value="1" />
+        <mass value="5" />
         <inertia
           ixx="1.0" ixy="0.0" ixz="0.0"
@@ -38,17 +38,17 @@
       <parent link="${prefix}_camera_mount" />
       <child link="${prefix}_camera_beam" />
-      <limit upper="1.57" lower="-1.57" velocity="0.3" effort="10"/>
+      <limit upper="1.57" lower="-1.57" velocity="10" effort="2"/>
        <axis xyz="0 0 1" />
     </joint>
     <transmission name="turret_trans">
-    <type>transmission_interface/SimpleTransmission</type>
-    <joint name="front_camera_pivot_joint">
-      <hardwareInterface>hardware_interface/PositionJointInterface</hardwareInterface>
-    </joint>
-    <actuator name="turret_motor">
-      <hardwareInterface>hardware_interface/PositionJointInterface</hardwareInterface>
-      <mechanicalReduction>1</mechanicalReduction>
-    </actuator>
-  </transmission>
+      <type>transmission_interface/SimpleTransmission</type>
+      <joint name="front_camera_pivot_joint">
+        <hardwareInterface>hardware_interface/PositionJointInterface</hardwareInterface>
+      </joint>
+      <actuator name="turret_motor">
+        <hardwareInterface>hardware_interface/PositionJointInterface</hardwareInterface>
+        <mechanicalReduction>1</mechanicalReduction>
+      </actuator>
+    </transmission>
     <gazebo reference="${prefix}_camera_beam">
       <material>Gazebo/DarkGrey</material>

Commit message: ns

File: src/ridgeback/ridgeback_description/urdf/accessories/camera_mount.urdf.xacro (robot description, xacro)
@@ -42,10 +42,10 @@
        <axis xyz="0 0 1" />
     </joint>
-    <transmission name="turret_trans">
+    <transmission name="{prefix}_turret_trans">
       <type>transmission_interface/SimpleTransmission</type>
-      <joint name="front_camera_pivot_joint">
+      <joint name="{prefix}_front_camera_pivot_joint">
         <hardwareInterface>hardware_interface/PositionJointInterface</hardwareInterface>
       </joint>
-      <actuator name="turret_motor">
+      <actuator name="{prefix}_turret_motor">
         <hardwareInterface>hardware_interface/PositionJointInterface</hardwareInterface>
         <mechanicalReduction>1</mechanicalReduction>

File: src/ridgeback/ridgeback_description/urdf/custom_sensors.urdf.xacro (robot description, xacro)
@@ -8,5 +8,5 @@
   <xacro:include filename="$(find lms1xx)/urdf/sick_lms1xx.urdf.xacro" />
   <xacro:macro name="sick_lms1xx_mount" params="prefix topic location">
-    <xacro:sick_lms1xx frame="${prefix}_laser" topic="${topic}" update_rate="50"  min_angle="-${M_PI}" max_angle="${M_PI}" />
+    <xacro:sick_lms1xx frame="${prefix}_laser" topic="${topic}" update_rate="50"  min_angle="-${M_PI}" max_angle="${M_PI}" robot_namespace="$(arg namespace)" />
     <joint name="${prefix}_laser_joint" type="fixed">
       <!-- This offset is from the base of the bracket to the LIDAR's focal point. -->

File: src/ridgeback/ridgeback_description/urdf/ridgeback.urdf.xacro (robot description, xacro)
@@ -1,4 +1,4 @@
 <?xml version="1.0"?>
-<robot name="ridgeback" xmlns:xacro="http://ros.org/wiki/xacro">
+<robot name="ridgeback" xmlns:xacro="http://www.ros.org/wiki/xacro">
   <xacro:property name="PI" value="3.1415926535897931" />
   <xacro:property name="wheel_radius" value="0.0759" />

Commit message: ns

File: src/ridgeback/ridgeback_description/urdf/accessories/camera_mount.urdf.xacro (robot description, xacro)
@@ -42,10 +42,10 @@
        <axis xyz="0 0 1" />
     </joint>
-    <transmission name="{prefix}_turret_trans">
+    <transmission name="turret_trans">
       <type>transmission_interface/SimpleTransmission</type>
-      <joint name="{prefix}_front_camera_pivot_joint">
+      <joint name="front_camera_pivot_joint">
         <hardwareInterface>hardware_interface/PositionJointInterface</hardwareInterface>
       </joint>
-      <actuator name="{prefix}_turret_motor">
+      <actuator name="turret_motor">
         <hardwareInterface>hardware_interface/PositionJointInterface</hardwareInterface>
         <mechanicalReduction>1</mechanicalReduction>

File: src/ridgeback/ridgeback_description/urdf/custom_sensors.urdf.xacro (robot description, xacro)
@@ -21,5 +21,5 @@
   <xacro:include filename="accessories/camera_mount.urdf.xacro" />
   <xacro:include filename="$(find pointgrey_camera_description)/urdf/pointgrey_flea3.urdf.xacro" />
-  <xacro:if value="$(optenv JACKAL_FLEA3 0)">
+  <xacro:if value="$(optenv JACKAL_FLEA3 1)">
     <camera_mount prefix="$(optenv JACKAL_FLEA_MOUNT front)"
                        tilt="$(optenv JACKAL_FLEA_TILT 0)"/>
