Commit message: change model from ridgeback to icra competition robot

File: src/pointgrey_camera_driver/pointgrey_camera_description/urdf/pointgrey_flea3.urdf.xacro (robot description, xacro)
@@ -9,19 +9,21 @@
       <inertial>
         <mass value="${camera_mass}" />
-        <inertia ixx="1e-6" ixy="0" ixz="0" iyy="1e-6" iyz="0" izz="1e-6" />
+      <inertia
+          ixx="0.0072228"
+          ixy="1.8624E-07"
+          ixz="5.1373E-07"
+          iyy="0.0035103"
+          iyz="-0.0016193"
+          izz="0.00443" />
       </inertial>
       <visual>
-        <origin xyz="0 0 0" rpy="0 0 0" />
+        <origin xyz="0 0 0.1" rpy="0 0 0" />
         <geometry>
-          <box size="${camera_x} ${camera_y} ${camera_z}"/>
+          <mesh filename="package://ridgeback_description/meshes/gun_new.STL"/>
         </geometry>
-        <material name="dark_grey" />
+        <material name="Black">
+          <color rgba="0.15 0.15 0.15 1.0"/>
+        </material>
       </visual>
-      <collision>
-        <origin xyz="0 0 0" rpy="0 0 0" />
-        <geometry>
-          <box size="${camera_x} ${camera_y} ${camera_z}" />
-        </geometry>
-      </collision>
     </link>
     <link name="${frame}_optical" />
@@ -33,5 +35,5 @@
     <!-- Gazebo -->
     <gazebo reference="${frame}_optical">
-      <material>Gazebo/Grey</material>
+      <material>Gazebo/Black</material>
       <sensor type="camera" name="${name}">
         <update_rate>${fps}</update_rate>
@@ -70,4 +72,7 @@
       </sensor>
     </gazebo>
+  <gazebo reference="${frame}">
+      <material>Gazebo/DarkGrey</material>
+  </gazebo>
   </xacro:macro>
 </robot>

File: src/ridgeback/ridgeback_description/urdf/accessories/camera_mount.urdf.xacro (robot description, xacro)
@@ -3,17 +3,19 @@
   <xacro:macro name="camera_mount" params="prefix tilt:=0">
     <link name="${prefix}_camera_mount">
-      <visual>
-        <origin xyz="0 0 0" rpy="1.5707 0 1.5707" />
-        <geometry>
-          <mesh filename="package://multi_jackal_description/meshes/camera-bracket.stl" scale="0.001 0.001 0.001" />
-        </geometry>
-        <material name="dark_grey" />
-      </visual>
-      <collision>
-      <origin xyz="0 0 0" rpy="1.5707 0 1.5707" />
-      <geometry>
-          <mesh filename="package://multi_jackal_description/meshes/camera-bracket.stl" scale="0.001 0.001 0.001" />
-        </geometry>
-      </collision>
+<!--      <visual>-->
+<!--        <origin xyz="-0.1 -0.25 1" rpy="0 0 1.5707" />-->
+<!--          <origin xyz="0 0 0" rpy="1.5707 0 1.5707" />-->
+<!--        <geometry>-->
+<!--          <mesh filename="package://multi_jackal_description/meshes/camera-bracket.stl" scale="0.001 0.001 0.001" />-->
+<!--            <mesh filename="package://ridgeback_description/meshes/ICRA_gun.STL" scale="0.001 0.001 0.001"/>-->
+<!--        </geometry>-->
+<!--        <material name="dark_grey" />-->
+<!--      </visual>-->
+<!--      <collision>-->
+<!--      <origin xyz="0 0 0" rpy="1.5707 0 1.5707" />-->
+<!--      <geometry>-->
+<!--          <mesh filename="package://multi_jackal_description/meshes/camera-bracket.stl" scale="0.001 0.001 0.001" />-->
+<!--        </geometry>-->
+<!--      </collision>-->
       <inertial>
         <origin xyz="0 0 0" rpy="0 0 0" />
@@ -26,18 +28,22 @@
     </link>
     <link name="${prefix}_camera_beam">
-      <visual>
-        <origin xyz="0 0 0" rpy="0 0 1.5707" />
-        <geometry>
-          <mesh filename="package://multi_jackal_description/meshes/camera-beam.stl" scale="0.001 0.001 0.001" />
-        </geometry>
-        <material name="dark_grey" />
-      </visual>
+<!--      <visual>-->
+<!--        <origin xyz="-0.1 -0.25 1" rpy="1.5707 0 0" />-->
+<!--          <origin xyz="0 0 0" rpy="0 0 1.5707" />-->
+<!--        <geometry>-->
+<!--          <mesh filename="package://multi_jackal_description/meshes/camera-beam.stl" scale="0.001 0.001 0.001" />-->
+<!--          <mesh filename="package://ridgeback_description/meshes/ICRA_gun.STL" scale="0.001 0.001 0.001"/>-->
+<!--        </geometry>-->
+<!--        <material name="dark_grey" />-->
+<!--      </visual>-->
     </link>
     <joint name="${prefix}_camera_pivot_joint" type="revolute">
-      <origin xyz="0.102 0 0.008" rpy="0 ${tilt} 0" />
+<!--      <joint name="${prefix}_camera_pivot_joint" type="fixed">-->
+<!--      <origin xyz="-0.1 -0.25 0.07" rpy="0 0 0" />-->
+        <origin xyz="0.14 0.002 0.008" rpy="0 ${tilt} 0" />
       <parent link="${prefix}_camera_mount" />
       <child link="${prefix}_camera_beam" />
       <!-- this velocity variable determines whether the joint rotates fast or slow -->
-      <limit upper="1.57" lower="-1.57" velocity="10" effort="2"/>
+      <limit upper="1.5707" lower="-1.5707" velocity="10" effort="2"/>
        <axis xyz="0 0 1" />
     </joint>

File: src/ridgeback/ridgeback_description/urdf/custom_sensors.urdf.xacro (robot description, xacro)
@@ -10,5 +10,5 @@
     <xacro:sick_lms1xx frame="${prefix}_laser" topic="${topic}" update_rate="50"
                        min_angle="-${M_PI}" max_angle="${M_PI}"
-                       min_range="0.73" robot_namespace="$(arg namespace)" />
+                       min_range="0.78" robot_namespace="$(arg namespace)" />
     <joint name="${prefix}_laser_joint" type="fixed">
       <!-- This offset is from the base of the bracket to the LIDAR's focal point. -->
@@ -27,5 +27,5 @@
                        tilt="$(optenv JACKAL_FLEA_TILT 0)"/>
     <joint name="$(optenv JACKAL_FLEA3_MOUNT front)_camera_mount_joint" type="fixed">
-      <origin xyz="$(optenv JACKAL_FLEA3_OFFSET 0.1 0 0.32)"
+      <origin xyz="$(optenv JACKAL_FLEA3_OFFSET -0.13 -0.01 0.22)"
               rpy="$(optenv JACKAL_FLEA3_RPY 0 0 0)" />
       <parent link="$(optenv JACKAL_FLEA_MOUNT front)_cover_link" />
@@ -34,7 +34,7 @@
     <pointgrey_flea3 frame="$(optenv JACKAL_FLEA3_MOUNT front)_camera" name="$(optenv JACKAL_FLEA_NAME front)"
       camera_x="0.0754" camera_y="0.029" camera_z="0.035"
-      camera_mass="0.085" hfov="1.0471975512" fps="60" width="640" height="512"/>
+      camera_mass="0.98307" hfov="1.0471975512" fps="60" width="640" height="512"/>
     <joint name="$(optenv JACKAL_FLEA3_MOUNT front)_camera_bracket_joint" type="fixed">
-      <origin xyz="0.020 0 0.0245" rpy="0 0 0" />
+      <origin xyz="0 0 0" rpy="0 0 0" />
       <parent link="$(optenv JACKAL_FLEA3_MOUNT front)_camera_beam" />
       <child link="$(optenv JACKAL_FLEA3_MOUNT front)_camera" />

File: src/ridgeback/ridgeback_description/urdf/ridgeback.urdf.xacro (robot description, xacro)
@@ -2,13 +2,13 @@
 <robot name="ridgeback" xmlns:xacro="http://www.ros.org/wiki/xacro">
   <xacro:property name="PI" value="3.1415926535897931" />
-  <xacro:property name="wheel_radius" value="0.0759" />
-  <xacro:property name="wheel_width" value="0.0790" />
+  <xacro:property name="wheel_radius" value="0.07" />
+  <xacro:property name="wheel_width" value="0.04" />
   <xacro:property name="chassis_length" value="0.960" />
   <xacro:property name="chassis_width" value="0.793" />
-  <xacro:property name="chassis_height" value="0.216" />
+  <xacro:property name="chassis_height" value="0.212" />
   <xacro:property name="deck_height" value="0.280" />
   <xacro:property name="axle_offset" value="0.0500" />
-  <xacro:property name="rocker_offset" value="0.319" />
-  <xacro:property name="rocker_width" value="0.472" />
+  <xacro:property name="rocker_offset" value="0.212" />
+  <xacro:property name="rocker_width" value="0.402" />
   <xacro:property name="imu_offset_x" value="0.2085" />
   <xacro:property name="imu_offset_y" value="-0.2902" />
@@ -24,12 +24,12 @@
     <link name="${prefix}_${side}_wheel_link">
       <visual>
-        <origin xyz="0 0 0" rpy="${PI/2} 0 0"/>
+        <origin xyz="0 0 0" rpy="0 0 0"/>
         <geometry>
-          <mesh filename="package://ridgeback_description/meshes/wheel.stl"/>
+          <mesh filename="package://ridgeback_description/meshes/wheel_new.STL" />
         </geometry>
         <material name="black" />
       </visual>
       <collision>
-        <origin xyz="0 0 0" rpy="${PI/2} 0 0"/>
+        <origin xyz="0 -0.01 0" rpy="${PI/2} 0 0"/>
         <geometry>
           <cylinder radius="${wheel_radius}" length="${wheel_width}"/>
@@ -63,11 +63,4 @@
   <xacro:macro name="rocker" params="prefix joint_type location *joint_limits">
     <link name="${prefix}_rocker_link">
-      <visual>
-        <origin xyz="0 0 0" rpy="${PI/2} 0 ${PI/2}" />
-        <geometry>
-          <mesh filename="package://ridgeback_description/meshes/rocker.stl"/>
-        </geometry>
-        <material name="black" />
-      </visual>
       <inertial>
         <origin xyz="0 0 0" rpy="${PI/2} 0 ${PI/2}"/>
@@ -87,8 +80,8 @@
     </joint>
     <xacro:wheel prefix="${prefix}" side="left">
-      <origin xyz="0 ${rocker_width/2 + wheel_width/2} 0" rpy="0 0 0" />
+      <origin xyz="-0.005 0.21 0.03" rpy="0 0 0" />
     </xacro:wheel>
     <xacro:wheel prefix="${prefix}" side="right">
-      <origin xyz="0 ${-(rocker_width/2 + wheel_width/2)} 0" rpy="0 0 0" />
+      <origin xyz="-0.005 -0.18 0.03" rpy="0 0 0" />
     </xacro:wheel>
   </xacro:macro>
@@ -107,14 +100,14 @@
   <link name="chassis_link">
     <visual>
-      <origin xyz="0 0 0" rpy="0 0 0" />
+            <origin xyz=" 0 0 0" rpy="0 0 0" />
       <geometry>
-        <mesh filename="package://ridgeback_description/meshes/body.stl"/>
+        <mesh filename="package://ridgeback_description/meshes/body_version2.STL" />
       </geometry>
       <material name="black" />
     </visual>
     <collision>
-      <origin xyz="0 0 0"/>
-      <geometry>
-        <mesh filename="package://ridgeback_description/meshes/body-collision.stl"/>
+      <origin xyz="0 0 0.35" rpy="0 0 0" />
+      <geometry>-0.005
+        <box size="0.55 0.4 0.2" />
       </geometry>
     </collision>
@@ -129,30 +122,16 @@
   </link>
   <joint name="right_side_cover_link_joint" type="fixed">
-    <origin xyz="0 0 0" rpy="0 0 0" />
+    <origin xyz="-0.02 0 0.3" rpy="0 0 0" />
     <parent link="chassis_link"/>
     <child link="right_side_cover_link" />
   </joint>
   <joint name="left_side_cover_link_joint" type="fixed">
-    <origin xyz="0 0 0" rpy="0 0 0" />
+    <origin xyz="-0.02 0 0.18" rpy="0 0 0" />
     <parent link="chassis_link"/>
     <child link="left_side_cover_link" />
   </joint>
   <link name="left_side_cover_link">
-    <visual>
-      <origin xyz="0 0 0" rpy="0 0 ${PI}" />
-      <geometry>
-        <mesh filename="package://ridgeback_description/meshes/side-cover.stl"/>
-      </geometry>
-      <material name="yellow" />
-    </visual>
   </link>
   <link name="right_side_cover_link">
-    <visual>
-      <origin xyz="0 0 0" rpy="0 0 0" />
-      <geometry>
-        <mesh filename="package://ridgeback_description/meshes/side-cover.stl"/>
-      </geometry>
-      <material name="yellow" />
-    </visual>
   </link>
   <joint name="front_cover_link_joint" type="fixed">
@@ -162,11 +141,4 @@
   </joint>
   <link name="front_cover_link">
-    <visual>
-      <origin xyz="0 0 0" rpy="0 0 0" />
-      <geometry>
-        <mesh filename="package://ridgeback_description/meshes/end-cover.stl" />
-      </geometry>
-      <material name="black" />
-    </visual>
   </link>
   <joint name="rear_cover_link_joint" type="fixed">
@@ -176,11 +148,4 @@
   </joint>
   <link name="rear_cover_link">
-    <visual>
-      <origin xyz="0 0 0" rpy="0 0 ${PI}" />
-      <geometry>
-        <mesh filename="package://ridgeback_description/meshes/end-cover.stl" />
-      </geometry>
-      <material name="black" />
-    </visual>
   </link>
   <joint name="front_lights_link_joint" type="fixed">
@@ -195,40 +160,13 @@
   </joint>
   <link name="front_lights_link">
-    <visual>
-      <origin xyz="0 0 0" rpy="0 0 0" />
-      <geometry>
-        <mesh filename="package://ridgeback_description/meshes/lights.stl" />
-      </geometry>
-      <material name="white" />
-    </visual>
   </link>
   <link name="rear_lights_link">
-    <visual>
-      <origin xyz="0 0 0" rpy="0 0 ${PI}" />
-      <geometry>
-        <mesh filename="package://ridgeback_description/meshes/lights.stl" />
-      </geometry>
-      <material name="red" />
-    </visual>
   </link>
   <joint name="top_link_joint" type="fixed">
-    <origin xyz="0 0 0" rpy="0 0 0" />
+    <origin xyz="0 0 0.5" rpy="0 0 0" />
     <parent link="chassis_link"/>
     <child link="top_link" />
   </joint>
   <link name="top_link">
-    <visual>
-      <origin xyz="0 0 0" rpy="0 0 0" />
-      <geometry>
-        <mesh filename="package://ridgeback_description/meshes/top.stl" />
-      </geometry>
-      <material name="black" />
-    </visual>
-    <collision>
-      <origin xyz="0 0 0" rpy="0 0 0" />
-      <geometry>
-        <mesh filename="package://ridgeback_description/meshes/top.stl"/>
-      </geometry>
-    </collision>
   </link>
   <joint name="axle_joint" type="fixed">
@@ -238,11 +176,4 @@
   </joint>
   <link name="axle_link">
-    <visual>
-      <origin xyz="0 0 0" rpy="0 ${PI/2} 0" />
-      <geometry>
-        <mesh filename="package://ridgeback_description/meshes/axle.stl" />
-      </geometry>
-      <material name="black" />
-    </visual>
   </link>
   <link name="imu_link">
