Commit message: combine RoboRTS with ridgeback

File: src/ridgeback/ridgeback_description/urdf/custom_sensors.urdf.xacro (robot description, xacro)
@@ -8,8 +8,8 @@
   <xacro:include filename="$(find lms1xx)/urdf/sick_lms1xx.urdf.xacro" />
   <xacro:macro name="sick_lms1xx_mount" params="prefix topic location">
-    <xacro:sick_lms1xx frame="${prefix}_laser" topic="${topic}" update_rate="20"  min_angle="-${M_PI}" max_angle="${M_PI}" />
+    <xacro:sick_lms1xx frame="${prefix}_laser" topic="${topic}" update_rate="50"  min_angle="-${M_PI}" max_angle="${M_PI}" />
     <joint name="${prefix}_laser_joint" type="fixed">
       <!-- This offset is from the base of the bracket to the LIDAR's focal point. -->
-      <origin xyz="${location * 0.3999} 0 0.32" rpy="0 0 0" />
+      <origin xyz="${location * 0.3999} 0 0.3" rpy="0 0 0" />
       <parent link="chassis_link" />
       <child link="${prefix}_laser" />

Commit message: add monocular camera to robot model

File: src/ridgeback/ridgeback_description/urdf/custom_sensors.urdf.xacro (robot description, xacro)
@@ -19,3 +19,23 @@
                              topic="scan"
                              location="0" />
+  <xacro:include filename="accessories/camera_mount.urdf.xacro" />
+  <xacro:include filename="$(find pointgrey_camera_description)/urdf/pointgrey_flea3.urdf.xacro" />
+  <xacro:if value="$(optenv JACKAL_FLEA3 0)">
+    <camera_mount prefix="$(optenv JACKAL_FLEA_MOUNT front)"
+                       tilt="$(optenv JACKAL_FLEA_TILT 0)"/>
+    <joint name="$(optenv JACKAL_FLEA3_MOUNT front)_camera_mount_joint" type="fixed">
+      <origin xyz="$(optenv JACKAL_FLEA3_OFFSET 0.1 0 0.32)"
+              rpy="$(optenv JACKAL_FLEA3_RPY 0 0 0)" />
+      <parent link="$(optenv JACKAL_FLEA_MOUNT front)_cover_link" />
+      <child link="$(optenv JACKAL_FLEA_MOUNT front)_camera_mount" />
+    </joint>
+    <pointgrey_flea3 frame="$(optenv JACKAL_FLEA3_MOUNT front)_camera" name="$(optenv JACKAL_FLEA_NAME front)"
+      camera_x="0.0754" camera_y="0.029" camera_z="0.035"
+      camera_mass="0.085" hfov="1.0471975512" fps="60" width="640" height="512"/>
+    <joint name="$(optenv JACKAL_FLEA3_MOUNT front)_camera_bracket_joint" type="fixed">
+      <origin xyz="0.020 0 0.0245" rpy="0 0 0" />
+      <parent link="$(optenv JACKAL_FLEA3_MOUNT front)_camera_beam" />
+      <child link="$(optenv JACKAL_FLEA3_MOUNT front)_camera" />
+    </joint>
+  </xacro:if>
 </robot>

Commit message: update planner footprint, modify lidar min range, simplify robot model

File: src/ridgeback/ridgeback_description/urdf/custom_sensors.urdf.xacro (robot description, xacro)
@@ -8,7 +8,7 @@
   <xacro:include filename="$(find lms1xx)/urdf/sick_lms1xx.urdf.xacro" />
   <xacro:macro name="sick_lms1xx_mount" params="prefix topic location">
-    <xacro:sick_lms1xx frame="${prefix}_laser" topic="${topic}" update_rate="50"
+    <xacro:sick_lms1xx frame="${prefix}_laser" topic="${topic}" update_rate="20"
                        min_angle="-${M_PI}" max_angle="${M_PI}"
-                       min_range="0.78" robot_namespace="$(arg namespace)" />
+                       min_range="0.45" robot_namespace="$(arg namespace)" />
     <joint name="${prefix}_laser_joint" type="fixed">
       <!-- This offset is from the base of the bracket to the LIDAR's focal point. -->

File: src/ridgeback/ridgeback_description/urdf/ridgeback.urdf.xacro (robot description, xacro)
@@ -109,5 +109,5 @@
       <origin xyz="0 0 0.35" rpy="0 0 0" />
       <geometry>-0.005
-        <box size="0.55 0.4 0.2" />
+        <box size="0.55 0.44 0.2" />
       </geometry>
     </collision>

Commit message: add a camera_visualtag link
for robomaster visualtag

File: src/ridgeback/ridgeback_description/urdf/custom_sensors.urdf.xacro (robot description, xacro)
@@ -41,3 +41,11 @@
     </joint>
   </xacro:if>
+  <link name="camera_visualtag">
+  </link>
+  <joint name="visualtag_joint" type="fixed">
+    <origin xyz="0 0 0"
+            rpy="-1.57 0 -1.57" />
+    <parent link="front_camera" />
+    <child link="camera_visualtag" />
+  </joint>
 </robot>

Commit message: add enable/disable camera and turret config

File: src/ridgeback/ridgeback_description/urdf/custom_sensors.urdf.xacro (robot description, xacro)
@@ -21,7 +21,7 @@
                              topic="scan"
                              location="0" />
+  <xacro:if value="$(optenv JACKAL_FLEA3 1)">
   <xacro:include filename="accessories/camera_mount.urdf.xacro" />
   <xacro:include filename="$(find pointgrey_camera_description)/urdf/pointgrey_flea3.urdf.xacro" />
-  <xacro:if value="$(optenv JACKAL_FLEA3 1)">
     <camera_mount prefix="$(optenv JACKAL_FLEA_MOUNT front)"
                        tilt="$(optenv JACKAL_FLEA_TILT 0)"/>
@@ -40,5 +40,4 @@
       <child link="$(optenv JACKAL_FLEA3_MOUNT front)_camera" />
     </joint>
-  </xacro:if>
   <link name="camera_visualtag">
   </link>
@@ -46,6 +45,7 @@
     <origin xyz="0 0 0"
             rpy="-1.57 0 -1.57" />
-    <parent link="front_camera" />
+    <parent link="$(optenv JACKAL_FLEA3_MOUNT front)_camera" />
     <child link="camera_visualtag" />
   </joint>
+  </xacro:if>
 </robot>
